File: PLCC-32-To-DIP-28.kicad_pcb (KiCad board)
At the start: 2 copper layers, 36.8 x 19 mm, 4 parts, among them U1 27512, U2 27C512PLCC

Commit message: Fixed gerber settings. Gerber output
Other:
- rule pad_to_mask_clearance: 0 -> 0.1016
Changed lines of the file:
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@@
     (links 30)
     (no_connects 0)
-    (area 130.124999 95.834999 167.055001 114.985001)
+    (area 130.124999 95.834999 179.45 126.5682)
     (thickness 1.6)
     (drawings 12)
@@
     (pad_size 1.55 1.55)
     (pad_drill 1)
-    (pad_to_mask_clearance 0)
-    (aux_axis_origin 0 0)
+    (pad_to_mask_clearance 0.1016)
+    (aux_axis_origin 130.175 114.935)
     (visible_elements FFFFFF7F)
     (pcbplotparams
-      (layerselection 3178497)
+      (layerselection 283148289)
       (usegerberextensions true)
       (excludeedgelayer true)
@@
       (viasonmask false)
       (mode 1)
-      (useauxorigin false)
+      (useauxorigin true)
       (hpglpennumber 1)
       (hpglpenspeed 20)
@@
       (plotinvisibletext false)
       (padsonsilk false)
-      (subtractmaskfromsilk false)
+      (subtractmaskfromsilk true)
       (outputformat 1)
       (mirror false)
-      (drillshape 1)
+      (drillshape 0)
       (scaleselection 1)
-      (outputdirectory ""))
+      (outputdirectory gerbers/))
   )
   (net 0 "")
